File: kicad/ice30lp384_dev_board.kicad_pcb (KiCad board)
At the start: 2 copper layers, 12.7 x 21.3 mm, 15 parts, among them J1 Conn_01x08, J2 Conn_01x08, U1 MIC5365-1.2YC5-TR, U2 ECS-TXO-2520-33-250-AN-TR, U3 ICE40LP384-SG32, U4 W25X10CLSNIG

Commit message: Improved castellation compatibility
Improved compatibility with OshPark's castellation rules which involved changing all pin header pads to be round.
Cleaned up schematic.
Parts:
- J1, J2: footprint Connector_PinHeader_2.54mm:PinHeader_1x08_P2.54mm_Vertical -> nezbyte:PinHeader_1x08_P2.54mm_Vertical
Connections:
- net Net-(J1-Pad3) renamed IO_1
- net Net-(J1-Pad4) renamed IO_2
- net Net-(J1-Pad5) renamed IO_3
- net Net-(J1-Pad6) renamed IO_4
- net Net-(J1-Pad7) renamed IO_5
- net Net-(J1-Pad8) renamed IO_32
